File: electronics/sensor/carga-sensor.kicad_sch (KiCad schematic)
At the start: 74 parts, among them J1 USB2UART, J2 1.47 IPS LCD, J3 ConnBattery, J4 RTD_PT100, Q1 SS8050, Q2 SS8050, Q3 SS8050, SW1 RST, SW2 IN1, SW3 Boot, SW4 IN2, SW5 IN4, SW6 IN4, SW7 IN5, U1 CH340C, U2 ESP32-S3-WROOM-1, U3 TPS63001_SEPIC_3V3, U4 MAX31865xTP, U5 BQ24075RGT_DPPM, U6 HX711

Commit message: feat: create hx711 module schematic
Parts:
- removed C1, C12, C18, C19, C2, C20, C3, C4, C5, C6, C7, C8, C9: 100nF, Capacitor_SMD:C_0805_2012Metric_Pad1.18x1.45mm_HandSolder, symbol Device:C
- removed C10: 22uF, Capacitor_SMD:C_0805_2012Metric_Pad1.18x1.45mm_HandSolder, symbol Device:C
- removed C11, C15: 1uF, Capacitor_SMD:C_0805_2012Metric_Pad1.18x1.45mm_HandSolder, symbol Device:C
- removed C13, C16, C17: 10uF, Capacitor_SMD:C_0805_2012Metric_Pad1.18x1.45mm_HandSolder, symbol Device:C
- removed C14: 0.1uF, Capacitor_SMD:C_0805_2012Metric_Pad1.18x1.45mm_HandSolder, symbol Device:C
- removed C22, C23: 4.7uF, Capacitor_SMD:C_0805_2012Metric_Pad1.18x1.45mm_HandSolder, symbol Device:C
- removed D1: INDICATOR, LED_SMD:LED_1206_3216Metric_Pad1.42x1.75mm_HandSolder, symbol Device:LED
- removed D2: VDD, LED_SMD:LED_1206_3216Metric_Pad1.42x1.75mm_HandSolder, symbol Device:LED
- removed D3: green, LED_SMD:LED_0805_2012Metric_Pad1.15x1.40mm_HandSolder, symbol Device:LED
- removed D4: red, LED_SMD:LED_0805_2012Metric_Pad1.15x1.40mm_HandSolder, symbol Device:LED
- removed J1: USB2UART, Connector_USB:USB_C_Receptacle_GCT_USB4110, symbol Connector:USB_C_Receptacle_USB2.0_14P
- removed J2: 1.47 IPS LCD, Connector_PinHeader_2.54mm:PinHeader_1x08_P2.54mm_Vertical, symbol Connector_Generic:Conn_01x08
- removed J3: ConnBattery, Connector_PinHeader_2.54mm:PinHeader_1x03_P2.54mm_Vertical, symbol Connector_Generic:Conn_01x03
- removed J4: RTD_PT100, TerminalBlock_Phoenix:TerminalBlock_Phoenix_PT-1,5-3-5.0-H_1x03_P5.00mm_Horizontal, symbol Connector:Screw_Terminal_01x03
- removed JP1: 3_OR_2_Wire, Jumper:SolderJumper-3_P1.3mm_Open_RoundedPad1.0x1.5mm, symbol Jumper:SolderJumper_3_Open
- removed JP2: 2_Wire, Jumper:SolderJumper-2_P1.3mm_Open_TrianglePad1.0x1.5mm, symbol Jumper:SolderJumper_2_Open
- removed L1: 22uH 1A, Inductor_SMD:L_Bourns_SRP7028A_7.3x6.6mm, symbol Device:L
- removed Q1, Q2, Q3: SS8050, Package_TO_SOT_SMD:SOT-23_Handsoldering, symbol Transistor_BJT:BC817
- removed R1, R10, R13, R14, R2, R3, R4, R7, R8, R9: 1k, Resistor_SMD:R_0805_2012Metric_Pad1.20x1.40mm_HandSolder, symbol Device:R_US
- removed R11, R12: 10k, Resistor_SMD:R_0805_2012Metric_Pad1.20x1.40mm_HandSolder, symbol Device:R_US
- removed R15: 100, Resistor_SMD:R_0805_2012Metric_Pad1.20x1.40mm_HandSolder, symbol Device:R_US
- removed R16: 46.4K, Resistor_SMD:R_0805_2012Metric_Pad1.20x1.40mm_HandSolder, symbol Device:R_US
- removed R17: 2K2, Resistor_SMD:R_0805_2012Metric_Pad1.20x1.40mm_HandSolder, symbol Device:R_US
- removed R18: 1.13k, Resistor_SMD:R_0805_2012Metric_Pad1.20x1.40mm_HandSolder, symbol Device:R_US
- removed R19: 400 1%, Resistor_SMD:R_0805_2012Metric_Pad1.20x1.40mm_HandSolder, symbol Device:R_US
- removed R20, R21: 1K5, Resistor_SMD:R_0805_2012Metric_Pad1.20x1.40mm_HandSolder, symbol Device:R_US
- removed R5, R6: 5K1, Resistor_SMD:R_0805_2012Metric_Pad1.20x1.40mm_HandSolder, symbol Device:R_US
- removed SW1: RST, Button_Switch_SMD:SW_SPST_PTS810, symbol Switch:SW_Push
- removed SW2: IN1, Button_Switch_SMD:SW_SPST_Omron_B3FS-100xP, symbol Switch:SW_Push
- removed SW3: Boot, Button_Switch_SMD:SW_SPST_PTS810, symbol Switch:SW_Push
- removed SW4: IN2, Button_Switch_SMD:SW_SPST_Omron_B3FS-100xP, symbol Switch:SW_Push
- removed SW5, SW6: IN4, Button_Switch_SMD:SW_SPST_Omron_B3FS-100xP, symbol Switch:SW_Push
- removed SW7: IN5, Button_Switch_SMD:SW_SPST_Omron_B3FS-100xP, symbol Switch:SW_Push
- removed U1: CH340C, Package_SO:SOIC-16_3.9x9.9mm_P1.27mm, symbol Interface_USB:CH340C
- removed U2: ESP32-S3-WROOM-1, RF_Module:ESP32-S3-WROOM-1, symbol RF_Module:ESP32-S3-WROOM-1
- removed U3: TPS63001_SEPIC_3V3, Package_SON:Texas_DRC0010J_ThermalVias, symbol Regulator_Switching:TPS63001
- removed U4: MAX31865xTP, Package_DFN_QFN:TQFN-20-1EP_5x5mm_P0.65mm_EP3.25x3.25mm, symbol Sensor_Temperature:MAX31865xTP
- removed U5: BQ24075RGT_DPPM, Package_DFN_QFN:VQFN-16-1EP_3x3mm_P0.5mm_EP1.6x1.6mm, symbol Battery_Management:BQ24075RGT
- removed U6: HX711, Package_SO:SOIC-16_3.9x9.9mm_P1.27mm, symbol Analog_ADC:HX711
- added C21, C24: 20pF, Capacitor_SMD:C_0805_2012Metric_Pad1.18x1.45mm_HandSolder, symbol Device:C
- added C25: 10uF, Capacitor_SMD:C_0805_2012Metric_Pad1.18x1.45mm_HandSolder, symbol Device:C
- added C26: 100nF, Capacitor_SMD:C_0805_2012Metric_Pad1.18x1.45mm_HandSolder, symbol Device:C
- added J5: SensorConn, Connector_IDC:IDC-Header_2x05_P2.54mm_Vertical, symbol Connector_Generic:Conn_02x05_Odd_Even
- added J6: LoadCellConnB, TerminalBlock_Phoenix:TerminalBlock_Phoenix_PT-1,5-4-5.0-H_1x04_P5.00mm_Horizontal, symbol Connector:Screw_Terminal_01x04
- added J7: LoadCellConnA, TerminalBlock_Phoenix:TerminalBlock_Phoenix_PT-1,5-4-5.0-H_1x04_P5.00mm_Horizontal, symbol Connector:Screw_Terminal_01x04
- added Q4: SS8550, Package_TO_SOT_SMD:SOT-23, symbol Transistor_BJT:SS8550
- added R22: 10k, Resistor_SMD:R_0805_2012Metric_Pad1.20x1.40mm_HandSolder, symbol Device:R_US
- added R23: 24.4k, Resistor_SMD:R_0805_2012Metric_Pad1.20x1.40mm_HandSolder, symbol Device:R_US
- added U7: HX711, Package_SO:SOIC-16_3.9x9.9mm_P1.27mm, symbol Analog_ADC:HX711
- added Y1: 16Mhz, Crystal:Crystal_HC49-U_Vertical, symbol Device:Crystal
Connections:
- net +3.3V: now also J5.1 (Pin_1), U7.15 (RATE), U7.16 (DVDD)
- net GND: now also C21.2, C24.2, C25.2, C26.2, J5.10 (Pin_10), J6.4 (Pin_4), J7.4 (Pin_4), R23.2, U7.5 (AGND)
- new net: C24.1, U7.13 (XO), Y1.1
- new net: C21.1, U7.14 (XI), Y1.2
- new net: Q4.1 (B), U7.2 (BASE)
- new net: R22.2, R23.1, U7.4 (VFB)
- new net: C26.1, U7.6 (VBG)
- new net +5V: J5.2 (Pin_2), Q4.2 (E), U7.1 (VSUP)
- new net AVDD: C25.1, J6.3 (Pin_3), J7.3 (Pin_3), Q4.3 (C), R22.1, U7.3 (AVDD)
- new net DOUT: J5.4 (Pin_4), U7.12 (DOUT)
- new net INA+: J7.1 (Pin_1), U7.8 (INA+)
- new net INA-: J7.2 (Pin_2), U7.7 (INA-)
- new net INB+: J6.1 (Pin_1), U7.10 (INB+)
- new net INB-: J6.2 (Pin_2), U7.9 (INB-)
- new net PD_SCK: J5.6 (Pin_6), U7.11 (PD_SCK)
- no-connect marks 24 -> 0
Other:
- note added: "AVDD = VBG + ([R1 + R2] / R1) 4.3 = 1.25 + ([R1 + R2] / R1) 2.44 R1 = R2 R1 = 10K R2 = 2.44 R1 = 24.4K"
- note added: "RATE (digital input) 0 -> 10hz 1 -> 80Hz"
- note removed: "3 Wire to Force+ 2/4 Wire to GND Connect 2_Wire if use 2/4 Wire"
- note removed: "DPPM"
- note removed: "ESP32-S3-WROOM-1"
- note removed: "GND VCC SCL SDA RES DC CS BLK"
- note removed: "Program Fast-Charge Safety Timer (TMR): RTMR = tMAXCHG / (10 × KTMR ) KTMR = 48 s/kΩ from the electrical characteristics table. RTMR = (6.25 hr × 3600 s/hr) / (10 × 48 s/kΩ) = 46.8 kΩ -> 46.4 kΩ"
- note removed: "Program the Fast Charge Current (ISET): RISET = KISET / ICHG KISET = 890 AΩ from the electrical characteristics table. RISET = 890 AΩ / 0.8 A = 1.1125 kΩ -> 1.13 kΩ"
- note removed: "SEPIC 3.3V"
- note removed: "dynamic power path management"
- note removed: "miso - Also known as q, this is the input of the serial stream into the ESP32 mosi - Also known as d, this is the output of the serial stream from the ESP32 sclk - Clock signal. Each data bit is clocked out or in on the positive or negative edge of this signal quadwp - Write Protect signal. Only used for 4-bit (qio/qout) transactions. quadhd - Hold signal. Only used for 4-bit (qio/qout) transacti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"
- title: (none) -> Carga HX711 Module
- moved on the sheet: H1, H2, H3, H4
